File: SteeringBoard.kicad_pcb (KiCad board)
At the start: 2 copper layers, 78 parts, among them J1 SWD, J10 Conn_01x01_Pin, J11 Conn_01x01_Pin, J12 Conn_01x01_Pin, J13 Conn_01x01_Pin, J14 Conn_01x01_Pin, J15 Conn_01x01_Pin, J2 Conn_01x01_Pin, J3 Conn_01x01_Pin, J4 Conn_01x01_Pin, J5 Conn_01x01_Pin, J6 Conn_01x01_Pin, J7 Conn_01x01_Pin, J8 Conn_01x01_Pin, J9 Conn_01x01_Pin, SW1 Reset, U1 STM32L431CBTx, U2 ISO1044BD, U3 CDSOT23-T24CAN, U4 TPS562231DRLR

Commit message: layout changes
Parts:
- removed F1, F2, F3, F4, F5: Fuse, Fuse:Fuse_0805_2012Metric
- added J16: Conn_01x02_Pin, UTSVT_Connectors:Molex_MicroFit3.0_1x2xP3.00mm_PolarizingPeg_Vertical, F.Cu at (218.0, 87.2)
- added U5: RO-123.3S, UTSVT_ICs:RI3_DC_Converter, B.Cu at (228.5, 92.0)
- C1, C10, C11, C12, C13, C14, C15, C2, C3, C4, C5, C6, C7, C8, C9: footprint Capacitor_SMD:C_0805_2012Metric -> Capacitor_SMD:C_0603_1608Metric
- D1, D2, D3, D4, D5, D6, D7, D8: footprint LED_SMD:LED_0805_2012Metric -> LED_SMD:LED_0603_1608Metric
- FB1, FB2: footprint Inductor_SMD:L_0805_2012Metric -> Inductor_SMD:L_0603_1608Metric
- J10, J11, J12, J13, J14, J15, J2, J3, J4, J5, J6, J7, J8, J9, TP1, TP2, TP4, TP5: footprint Connector_PinHeader_2.54mm:PinHeader_1x01_P2.54mm_Vertical -> TestPoint:TestPoint_Pad_D1.0mm
- R1, R10, R11, R12, R13, R14, R15, R16, R17, R2, R3, R4, R5, R6, R7, R8, R9: footprint Resistor_SMD:R_0805_2012Metric -> Resistor_SMD:R_0603_1608Metric
- TP3: footprint TestPoint:TestPoint_Pad_D1.5mm -> TestPoint:TestPoint_Pad_D1.0mm
- U1, U2: moved to B.Cu
- moved J8 120.8 mm to (264.8, 77.1)
- moved J6 120.0 mm to (258.0, 77.1)
- moved J11 117.3 mm to (261.2, 93.5), turned to 90 degrees
- moved J7 116.0 mm to (258.8, 93.5), turned to 90 degrees
- moved J15 115.4 mm to (264.0, 93.5), turned to 90 degrees
- moved J14 114.2 mm to (262.5, 77.1)
- moved J5 113.0 mm to (251.2, 74.5)
- moved J9 112.3 mm to (256.0, 93.5), turned to 90 degrees
- moved J10 112.0 mm to (255.2, 77.1)
- moved J12 111.6 mm to (260.2, 77.1)
- moved R6 110.9 mm to (264.0, 90.8), turned to -90 degrees
- moved J4 110.2 mm to (249.0, 74.5)
- moved R4 108.5 mm to (261.2, 90.8), turned to -90 degrees
- moved R1 106.6 mm to (258.8, 90.8), turned to 90 degrees
- moved J13 105.6 mm to (253.5, 93.5), turned to 90 degrees
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Connections:
- R1 pad 2: Net-(U1-PA0) -> GND
- R2 pad 1: /CRS_SET- -> GND
- R2 pad 2: Net-(U1-PA1) -> /CRS_SET-
- R4 pad 1: /REG- -> GND
- R4 pad 2: Net-(U1-PA2) -> /REG-
- R5 pad 1: /TSS- -> GND
- R5 pad 2: Net-(U1-PA3) -> /TSS-
- R6 pad 1: /HRN_PD- -> GND
- R6 pad 2: Net-(U1-PA4) -> /HRN_PD-
- U1 pad 10: Net-(U1-PA0) -> /RGEN_E-
- U1 pad 11: Net-(U1-PA1) -> /CRS_SET-
- U1 pad 12: Net-(U1-PA2) -> /REG-
- U1 pad 13: Net-(U1-PA3) -> /TSS-
- U1 pad 14: Net-(U1-PA4) -> /HRN_PD-
Routing:
- net +3.3V: track 0.00 -> 38.6 mm
- net Net-(D4-A): track 0.00 -> 1.92 mm
- net /TSS-: track 0.00 -> 1.92 mm
- net /RGEN_E-: track 0.00 -> 1.92 mm
- net /REG-: track 0.00 -> 1.92 mm
- net /CRS_SET-: track 0.00 -> 1.92 mm
- net Net-(D2-A): track 0.00 -> 1.89 mm
- net Net-(D1-A): track 0.00 -> 1.89 mm
- net Net-(D7-A): track 0.00 -> 1.89 mm
- net Net-(D5-A): track 0.00 -> 1.89 mm
- net Net-(D3-A): track 0.00 -> 1.89 mm
- net /NRST: track 0.00 -> 1.88 mm
- added copper zone on F.Cu, net GND
- added copper zone on F.Cu, net GNDPWR
Other:
- board outline added: 59 x 26 mm

Commit message: Finished layout
Parts:
- C12, R12, SW1, U4: moved to B.Cu
- C2: value 100nF -> 300nF
- L1: footprint Inductor_SMD:L_0805_2012Metric_Pad1.15x1.40mm_HandSolder -> Inductor_SMD:L_0603_1608Metric; moved to B.Cu
- moved J4 102.7 mm to (147.8, 91.8)
- moved J15 101.3 mm to (163.2, 104.2)
- moved R6 101.3 mm to (163.2, 101.4)
- moved R12 97.5 mm to (133.8, 87.8)
- moved U3 97.3 mm to (137.8, 88.0)
- moved J2 97.3 mm to (141.5, 89.5)
- moved J3 96.9 mm to (141.5, 87.0)
- moved R13 95.4 mm to (141.9, 98.0)
- moved R14 95.4 mm to (138.4, 98.0)
- moved C12 94.6 mm to (133.2, 96.5), turned to 90 degrees
- moved J11 94.1 mm to (167.8, 104.2)
- moved R4 94.1 mm to (167.8, 101.4)
- moved C6 93.7 mm to (178.0, 98.5)
- moved C8 93.7 mm to (178.0, 95.0)
- moved C3 93.7 mm to (178.0, 96.8)
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Routing:
- net +3.3V: track 38.6 -> 102.7 mm, vias 0 -> 5
- net /NRST: track 1.88 -> 42.1 mm, vias 0 -> 1
- net GND: track 0.00 -> 38.0 mm, vias 0 -> 5
- net /CAN_RX: track 0.00 -> 30.7 mm, vias 0 -> 3
- net +12V: track 0.00 -> 30.3 mm, vias 0 -> 1
- net /SWDIO: track 0.00 -> 22.3 mm, vias 0 -> 2
- net /CAN_L: track 0.00 -> 16.8 mm, vias 0 -> 1
- net /SWCLK: track 0.00 -> 16.2 mm
- net /CAN_H: track 0.00 -> 15.0 mm, vias 0 -> 2
- net /3V3_Bus: track 0.00 -> 14.8 mm, vias 0 -> 2
- net GNDA: track 0.00 -> 14.1 mm, vias 0 -> 1
- net VDDA: track 0.00 -> 13.0 mm, vias 0 -> 1
- net /PowerDist/FB: track 0.00 -> 10.9 mm, vias 0 -> 1
- net /HRN_PD-: track 0.00 -> 7.93 mm, vias 0 -> 1
- net GNDPWR: track 0.00 -> 6.99 mm, vias 0 -> 4
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
Commit message: board update
Parts:
- added J17: Conn_01x01_Pin, TestPoint:TestPoint_Pad_D1.0mm, F.Cu at (158.8, 104.8)
Connections:
- U1 pad 19: /PB1 -> unconnected-(U1-PB1-Pad19)
- U1 pad 20: /PB2 -> unconnected-(U1-PB2-Pad20)
- U1 pad 39: /PB3 -> unconnected-(U1-PB3-Pad39)
- U1 pad 40: /PB4 -> unconnected-(U1-PB4-Pad40)
- U1 pad 41: /PB5 -> unconnected-(U1-PB5-Pad41)
- U1 pad 46: unconnected-(U1-PB9-Pad46) -> /CAN_TX
Changed lines of the file:
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@@
 	(net 37 "unconnected-(U1-PA8-Pad29)")
 	(net 38 "unconnected-(U1-PA15-Pad38)")
-	(net 39 "/PB5")
+	(net 39 "unconnected-(U1-PB5-Pad41)")
 	(net 40 "unconnected-(U1-PA6-Pad16)")
 	(net 41 "unconnected-(U1-VBAT-Pad1)")
 	(net 42 "unconnected-(U1-PH1-Pad6)")
 	(net 43 "/CAN_RX")
-	(net 44 "unconnected-(U1-PB9-Pad46)")
-	(net 45 "/PB2")
-	(net 46 "/PB4")
+	(net 44 "unconnected-(U1-PB2-Pad20)")
+	(net 45 "unconnected-(U1-PB4-Pad40)")
+	(net 46 "unconnected-(U1-PB3-Pad39)")
 	(net 47 "unconnected-(U1-PB12-Pad25)")
 	(net 48 "unconnected-(U1-PB13-Pad26)")
@@
 	(net 58 "unconnected-(U1-PB15-Pad28)")
 	(net 59 "unconnected-(U1-PB0-Pad18)")
-	(net 60 "/PB3")
+	(net 60 "unconnected-(U1-PB1-Pad19)")
 	(net 61 "unconnected-(U1-PB10-Pad21)")
 	(net 62 "unconnected-(U1-PB7-Pad43)")
-	(net 63 "/PB1")
-	(net 64 "/CAN_TX")
+	(net 63 "/CAN_TX")
 	(footprint "TestPoint:TestPoint_Pad_D1.0mm"
 		(layer "F.Cu")
@@
 			(size 1 1)
 			(layers "F.Cu" "F.Mask")
-			(net 64 "/CAN_TX")
+			(net 63 "/CAN_TX")
+			(pinfunction "Pin_1")
+			(pintype "passive")
+		)
+	)
+	(footprint "TestPoint:TestPoint_Pad_D1.0mm"
+		(layer "F.Cu")
+		(at 158.75 104.75)
+		(descr "SMD pad as test Point, diameter 1.0mm")
+		(tags "test point SMD pad")
+		(property "Reference" "J17"
+			(at 0 -1.448 0)
+			(layer "F.SilkS")
+			(effects
+				(font
+					(size 1 1)
+					(thickness 0.15)
+				)
+			)
+		)
+		(property "Value" "Conn_01x01_Pin"
+			(at 0 1.55 0)
+			(layer "F.Fab")
+			(effects
+				(font
+					(size 1 1)
+					(thickness 0.15)
+				)
+			)
+		)
+		(property "Footprint" "TestPoint:TestPoint_Pad_D1.0mm"
+			(at 0 0 0)
+			(unlocked yes)
+			(layer "F.Fab")
+			(hide yes)
+			(effects
+				(font
+					(size 1.27 1.27)
+					(thickness 0.15)
+				)
+			)
+		)
+		(property "Datasheet" ""
+			(at 0 0 0)
+			(unlocked yes)
+			(layer "F.Fab")
+			(hide yes)
+			(effects
+				(font
+					(size 1.27 1.27)
+					(thickness 0.15)
+				)
+			)
+		)
+		(property "Description" "Generic connector, single row, 01x01, script generated"
+			(at 0 0 0)
+			(unlocked yes)
+			(layer "F.Fab")
+			(hide yes)
+			(effects
+				(font
+					(size 1.27 1.27)
+					(thickness 0.15)
+				)
+			)
+		)
+		(property ki_fp_filters "Connector*:*_1x??_*")
+		(sheetname "Root")
+		(sheetfile "SteeringBoard.kicad_sch")
+		(attr exclude_from_pos_files)
+		(fp_circle
+			(center 0 0)
+			(end 0 0.7)
+			(stroke
+				(width 0.12)
+				(type solid)
+			)
+			(fill none)
+			(layer "F.SilkS")
+		)
+		(fp_circle
+			(center 0 0)
+			(end 1 0)
+			(stroke
+				(width 0.05)
+				(type solid)
+			)
+			(fill none)
+			(layer "F.CrtYd")
+		)
+		(fp_text user "${REFERENCE}"
+			(at 0 -1.45 0)
+			(layer "F.Fab")
+			(effects
+				(font
+					(size 1 1)
+					(thickness 0.15)
+				)
+			)
+		)
+		(pad "1" smd circle
+			(at 0 0)
+			(size 1 1)
+			(layers "F.Cu" "F.Mask")
+			(net 31 "/12V_Ext")
 			(pinfunction "Pin_1")
 			(pintype "passive")
@@
 		)
 		(fp_text user "${REFERENCE}"
-			(at 0 0 360)
+			(at 0 0 0)
 			(layer "B.Fab")
 			(effects
@@
 			(net 55 "unconnected-(U1-PH0-Pad5)")
 			(pinfunction "PH0")
-			(pintype "bidirectional")
+			(pintype "bidirectional+no_connect")
 		)
 		(pad "6" smd roundrect
@@
 			(net 42 "unconnected-(U1-PH1-Pad6)")
 			(pinfunction "PH1")
-			(pintype "bidirectional")
+			(pintype "bidirectional+no_connect")
 		)
 		(pad "7" smd roundrect
@@
 			(net 36 "unconnected-(U1-PA5-Pad15)")
 			(pinfunction "PA5")
-			(pintype "bidirectional")
+			(pintype "bidirectional+no_connect")
 		)
 		(pad "16" smd roundrect
@@
 			(net 40 "unconnected-(U1-PA6-Pad16)")
 			(pinfunction "PA6")
-			(pintype "bidirectional")
+			(pintype "bidirectional+no_connect")
 		)
 		(pad "17" smd roundrect
@@
 			(net 57 "unconnected-(U1-PA7-Pad17)")
 			(pinfunction "PA7")
-			(pintype "bidirectional")
+			(pintype "bidirectional+no_connect")
 		)
 		(pad "18" smd roundrect
@@
 			(layers "B.Cu" "B.Paste" "B.Mask")
 			(roundrect_rratio 0.25)
-			(net 63 "/PB1")
+			(net 60 "unconnected-(U1-PB1-Pad19)")
 			(pinfunction "PB1")
-			(pintype "bidirectional")
+			(pintype "bidirectional+no_connect")
 		)
 		(pad "20" smd roundrect
@@
 			(layers "B.Cu" "B.Paste" "B.Mask")
 			(roundrect_rratio 0.25)
-			(net 45 "/PB2")
+			(net 44 "unconnected-(U1-PB2-Pad20)")
 			(pinfunction "PB2")
-			(pintype "bidirectional")
+			(pintype "bidirectional+no_connect")
 		)
 		(pad "21" smd roundrect
@@
 			(net 61 "unconnected-(U1-PB10-Pad21)")
 			(pinfunction "PB10")
-			(pintype "bidirectional")
+			(pintype "bidirectional+no_connect")
 		)
 		(pad "22" smd roundrect
@@
 			(net 54 "unconnected-(U1-PB11-Pad22)")
 			(pinfunction "PB11")
-			(pintype "bidirectional")
+			(pintype "bidirectional+no_connect")
 		)
 		(pad "23" smd roundrect
@@
 			(net 47 "unconnected-(U1-PB12-Pad25)")
 			(pinfunction "PB12")
-			(pintype "bidirectional")
+			(pintype "bidirectional+no_connect")
 		)
 		(pad "26" smd roundrect
@@
 			(net 48 "unconnected-(U1-PB13-Pad26)")
 			(pinfunction "PB13")
-			(pintype "bidirectional")
+			(pintype "bidirectional+no_connect")
 		)
 		(pad "27" smd roundrect
@@
 			(net 33 "unconnected-(U1-PB14-Pad27)")
 			(pinfunction "PB14")
-			(pintype "bidirectional")
+			(pintype "bidirectional+no_connect")
 		)
 		(pad "28" smd roundrect
@@
 			(net 58 "unconnected-(U1-PB15-Pad28)")
 			(pinfunction "PB15")
-			(pintype "bidirectional")
+			(pintype "bidirectional+no_connect")
 		)
 		(pad "29" smd roundrect
@@
 			(net 53 "/USART1_TX")
 			(pinfunction "PA9")
-			(pintype "bidirectional")
+			(pintype "bidirectional+no_connect")
 		)
 		(pad "31" smd roundrect
@@
 			(net 35 "/USART1_RX")
 			(pinfunction "PA10")
-			(pintype "bidirectional")
+			(pintype "bidirectional+no_connect")
 		)
 		(pad "32" smd roundrect
@@
 			(layers "B.Cu" "B.Paste" "B.Mask")
 			(roundrect_rratio 0.25)
-			(net 60 "/PB3")
+			(net 46 "unconnected-(U1-PB3-Pad39)")
 			(pinfunction "PB3")
-			(pintype "bidirectional")
+			(pintype "bidirectional+no_connect")
 		)
 		(pad "40" smd roundrect
@@
 			(layers "B.Cu" "B.Paste" "B.Mask")
 			(roundrect_rratio 0.25)
-			(net 46 "/PB4")
+			(net 45 "unconnected-(U1-PB4-Pad40)")
 			(pinfunction "PB4")
-			(pintype "bidirectional")
+			(pintype "bidirectional+no_connect")
 		)
 		(pad "41" smd roundrect
@@
 			(layers "B.Cu" "B.Paste" "B.Mask")
 			(roundrect_rratio 0.25)
-			(net 39 "/PB5")
+			(net 39 "unconnected-(U1-PB5-Pad41)")
 			(pinfunction "PB5")
-			(pintype "bidirectional")
+			(pintype "bidirectional+no_connect")
 		)
 		(pad "42" smd roundrect
@@
 			(net 51 "unconnected-(U1-PB6-Pad42)")
 			(pinfunction "PB6")
-			(pintype "bidirectional")
+			(pintype "bidirectional+no_connect")
 		)
 		(pad "43" smd roundrect
@@
 			(net 62 "unconnected-(U1-PB7-Pad43)")
 			(pinfunction "PB7")
-			(pintype "bidirectional")
+			(pintype "bidirectional+no_connect")
 		)
 		(pad "44" smd roundrect
@@
 			(layers "B.Cu" "B.Paste" "B.Mask")
 			(roundrect_rratio 0.25)
-			(net 44 "unconnected-(U1-PB9-Pad46)")
+			(net 63 "/CAN_TX")
 			(pinfunction "PB9")
 			(pintype "bidirectional")
@@
 			(layers "B.Cu" "B.Paste" "B.Mask")
 			(roundrect_rratio 0.25)
-			(net 64 "/CAN_TX")
+			(net 63 "/CAN_TX")
 			(pinfunction "TXD")
 			(pintype "input")
@@
 		(width 0.2)
 		(layer "F.Cu")
-		(net 64)
+		(net 63)
 	)
 	(segment
@@
 		(width 0.2)
 		(layer "F.Cu")
-		(net 64)
+		(net 63)
 	)
 	(via
@@
 		(drill 0.3)
 		(layers "F.Cu" "B.Cu")
-		(net 64)
+		(net 63)
 	)
 	(zone

Commit message: board update
Parts:
- moved C7 22.9 mm to (155.8, 84.5), turned to -90 degrees
- moved R3 21.7 mm to (157.5, 84.5), turned to -90 degrees
- moved FB1 20.7 mm to (159.2, 84.5), turned to 90 degrees
- moved C8 19.9 mm to (161.0, 84.5), turned to 90 degrees
- moved FB2 19.6 mm to (166.2, 84.5), turned to 90 degrees
- moved C3 19.6 mm to (162.8, 84.5), turned to 90 degrees
- moved C6 19.4 mm to (164.5, 84.5), turned to 90 degrees
- moved J5 13.0 mm to (146.8, 89.8)
- moved J17 11.5 mm to (147.5, 102.5)
- moved C15 11.2 mm to (152.2, 98.5)
- moved C9 11.2 mm to (149.5, 98.5)
- moved J11 8.17 mm to (159.8, 102.5)
- moved J13 8.17 mm to (157.5, 102.5)
- moved J15 8.17 mm to (155.2, 102.5)
- moved J7 8.17 mm to (164.2, 102.5)
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Connections:
- J17 pad 1: /12V_Ext -> +12V
- R3 pad 1: VDD -> +3.3V
- U1 pad 8: GNDA -> unconnected-(U1-VSSA-Pad8)
- U1 pad 9: VDDA -> unconnected-(U1-VDDA-Pad9)
Routing:
- net /CAN_RX: track 30.7 -> 0.00 mm, vias 3 -> 0
- net /SWDIO: track 22.3 -> 0.00 mm, vias 2 -> 0
- net /NRST: track 42.1 -> 23.6 mm, vias 1 -> 0
- net /SWCLK: track 16.2 -> 0.00 mm
- net +3.3V: track 102.7 -> 89.6 mm, vias 5 -> 4
- net GNDA: track 14.1 -> 5.26 mm
- net VDDA: track 13.0 -> 6.27 mm
- net /CAN_TX: track 3.20 -> 0.00 mm, vias 1 -> 0
Other:
- board size 59 x 26 mm -> 52 x 26 mm

Commit message: board update
Parts:
- removed D8: 12V, LED_SMD:LED_0603_1608Metric
- removed R17: 22.1k, Resistor_SMD:R_0603_1608Metric
- moved J17 9.17 mm to (139.2, 106.5)
- moved C9 6.35 mm to (152.2, 104.2), turned to 180 degrees
- moved C1 5.53 mm to (152.3, 97.0)
- moved C2 5.53 mm to (152.3, 95.2)
- moved C4 5.53 mm to (152.3, 98.8)
- moved C5 5.53 mm to (152.3, 100.5)
- moved J5 4.27 mm to (148.2, 93.8)
- moved C15 4.03 mm to (152.2, 102.5), turned to 180 degrees
- moved U1 3.34 mm to (156.0, 95.0)
- moved J4 2.55 mm to (148.2, 91.5)
- moved C6 0.07 mm to (164.5, 84.5)
- moved FB2 0.07 mm to (166.2, 84.5)
Routing:
- net /CAN_TX: track 0.00 -> 15.6 mm, vias 0 -> 2
- net /CAN_RX: track 0.00 -> 14.9 mm, vias 0 -> 2
- net /SWDIO: track 0.00 -> 14.9 mm
- net /NRST: track 23.6 -> 34.0 mm, vias 0 -> 1
- net GND: track 38.0 -> 48.0 mm, vias 5 -> 4
- net /SWCLK: track 0.00 -> 8.07 mm, vias 0 -> 2
- net /RGEN_E-: track 6.78 -> 10.3 mm
- net +12V: track 30.3 -> 27.8 mm
- net Net-(D8-A): track 2.42 -> 0.00 mm
- net /CRS_SET-: track 6.34 -> 8.39 mm
- net /TSS-: track 7.60 -> 5.78 mm
- net +3.3V: track 89.6 -> 90.9 mm
- net /REG-: track 7.54 -> 6.85 mm
- net /PowerDist/FB: track 10.9 -> 11.5 mm, vias 1 -> 3
- net VDDA: track 6.27 -> 5.91 mm, vias 1 -> 0
