File: CAN.kicad_sch (KiCad schematic)
At the start: 6 parts, among them U5 ISO1044BD, U6 CDSOT23-T24CAN

Commit message: scheme update
Parts:
- renumbered C21 to C10, C20 to C9, JP3 to JP1, R21 to R12, U5 to U2, U6 to U3
Changed lines of the file:
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@@
 		(on_board yes)
 		(dnp no)
-		(property "Reference" "C20"
+		(property "Reference" "C9"
 			(at 75.184 80.772 0)
 			(effects
@@
 			(project "SteeringBoard"
 				(path "/1bc9055e-ec57-4cc6-8fa0-537b054d5f7c/2ae31cd1-3b20-41d6-acf0-8556f0359c18"
-					(reference "C20")
+					(reference "C9")
 					(unit 1)
 				)
@@
 		(dnp no)
 		(fields_autoplaced yes)
-		(property "Reference" "U6"
+		(property "Reference" "U3"
 			(at 144.78 89.535 0)
 			(effects
@@
 			(project "SteeringBoard"
 				(path "/1bc9055e-ec57-4cc6-8fa0-537b054d5f7c/2ae31cd1-3b20-41d6-acf0-8556f0359c18"
-					(reference "U6")
+					(reference "U3")
 					(unit 1)
 				)
@@
 		(on_board yes)
 		(dnp no)
-		(property "Reference" "#PWR041"
+		(property "Reference" "#PWR027"
 			(at 74.93 78.74 0)
 			(effects
@@
 			(project "SteeringBoard"
 				(path "/1bc9055e-ec57-4cc6-8fa0-537b054d5f7c/2ae31cd1-3b20-41d6-acf0-8556f0359c18"
-					(reference "#PWR041")
+					(reference "#PWR027")
 					(unit 1)
 				)
@@
 		(dnp no)
 		(fields_autoplaced yes)
-		(property "Reference" "U5"
+		(property "Reference" "U2"
 			(at 102.87 71.755 0)
 			(effects
@@
 			(project "SteeringBoard"
 				(path "/1bc9055e-ec57-4cc6-8fa0-537b054d5f7c/2ae31cd1-3b20-41d6-acf0-8556f0359c18"
-					(reference "U5")
+					(reference "U2")
 					(unit 1)
 				)
@@
 		(dnp no)
 		(fields_autoplaced yes)
-		(property "Reference" "#PWR043"
+		(property "Reference" "#PWR029"
 			(at 154.94 87.63 0)
 			(effects
@@
 			(project "SteeringBoard"
 				(path "/1bc9055e-ec57-4cc6-8fa0-537b054d5f7c/2ae31cd1-3b20-41d6-acf0-8556f0359c18"
-					(reference "#PWR043")
+					(reference "#PWR029")
 					(unit 1)
 				)
@@
 		(on_board yes)
 		(dnp no)
-		(property "Reference" "R21"
+		(property "Reference" "R12"
 			(at 123.698 91.44 90)
 			(effects
@@
 			(project "SteeringBoard"
 				(path "/1bc9055e-ec57-4cc6-8fa0-537b054d5f7c/2ae31cd1-3b20-41d6-acf0-8556f0359c18"
-					(reference "R21")
+					(reference "R12")
 					(unit 1)
 				)
@@
 		(dnp no)
 		(fields_autoplaced yes)
-		(property "Reference" "#PWR044"
+		(property "Reference" "#PWR030"
 			(at 154.94 101.6 0)
 			(effects
@@
 			(project "SteeringBoard"
 				(path "/1bc9055e-ec57-4cc6-8fa0-537b054d5f7c/2ae31cd1-3b20-41d6-acf0-8556f0359c18"
-					(reference "#PWR044")
+					(reference "#PWR030")
 					(unit 1)
 				)
@@
 		(on_board yes)
 		(dnp no)
-		(property "Reference" "#PWR042"
+		(property "Reference" "#PWR028"
 			(at 74.93 93.98 0)
 			(effects
@@
 			(project "SteeringBoard"
 				(path "/1bc9055e-ec57-4cc6-8fa0-537b054d5f7c/2ae31cd1-3b20-41d6-acf0-8556f0359c18"
-					(reference "#PWR042")
+					(reference "#PWR028")
 					(unit 1)
 				)
@@
 		(on_board yes)
 		(dnp no)
-		(property "Reference" "C21"
+		(property "Reference" "C10"
 			(at 139.954 75.692 0)
 			(effects
@@
 			(project "SteeringBoard"
 				(path "/1bc9055e-ec57-4cc6-8fa0-537b054d5f7c/2ae31cd1-3b20-41d6-acf0-8556f0359c18"
-					(reference "C21")
+					(reference "C10")
 					(unit 1)
 				)
@@
 		(on_board yes)
 		(dnp no)
-		(property "Reference" "JP3"
+		(property "Reference" "JP1"
 			(at 120.65 97.028 0)
 			(effects
@@
 			(project "SteeringBoard"
 				(path "/1bc9055e-ec57-4cc6-8fa0-537b054d5f7c/2ae31cd1-3b20-41d6-acf0-8556f0359c18"
-					(reference "JP3")
-					(unit 1)
-				)
+					(reference "JP1")
+					(unit 1)
+				)

Commit message: layout changes
Parts:
- C10, C9: footprint Capacitor_SMD:C_0805_2012Metric -> Capacitor_SMD:C_0603_1608Metric
- R12: footprint Resistor_SMD:R_0805_2012Metric -> Resistor_SMD:R_0603_1608Metric
Changed lines of the file:
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@@
 			)
 		)
-		(property "Footprint" "Capacitor_SMD:C_0805_2012Metric"
+		(property "Footprint" "Capacitor_SMD:C_0603_1608Metric"
 			(at 74.93 82.55 0)
 			(effects
@@
 			)
 		)
-		(property "Footprint" "Resistor_SMD:R_0805_2012Metric"
+		(property "Footprint" "Resistor_SMD:R_0603_1608Metric"
 			(at 127.508 91.44 90)
 			(effects
@@
 			)
 		)
-		(property "Footprint" "Capacitor_SMD:C_0805_2012Metric"
+		(property "Footprint" "Capacitor_SMD:C_0603_1608Metric"
 			(at 139.7 77.47 0)
 			(effects

Commit message: finished board with ldo
Parts:
- renumbered C9 to C8, C10 to C9, R12 to R8
Other:
- moved on the sheet: JP1
Changed lines of the file:
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@@
+	(wire
+		(pts
+			(xy 125.73 97.79) (xy 125.73 95.25)
+		)
+		(stroke
+			(width 0)
+			(type default)
+		)
+	)
 	(wire
 		(pts
@@
 	(wire
 		(pts
-			(xy 125.73 99.06) (xy 125.73 95.25)
-		)
-		(stroke
-			(width 0)
-			(type default)
-		)
-	)
-	(wire
-		(pts
 			(xy 74.93 78.74) (xy 92.71 78.74)
 		)
@@
 	(wire
 		(pts
-			(xy 115.57 86.36) (xy 115.57 99.06)
+			(xy 115.57 86.36) (xy 115.57 97.79)
 		)
 		(stroke
@@
 		(on_board yes)
 		(dnp no)
-		(property "Reference" "C9"
+		(property "Reference" "C8"
 			(at 75.184 80.772 0)
 			(effects
@@
 			(project "SteeringBoard"
 				(path "/1bc9055e-ec57-4cc6-8fa0-537b054d5f7c/2ae31cd1-3b20-41d6-acf0-8556f0359c18"
-					(reference "C9")
+					(reference "C8")
 					(unit 1)
 				)
@@
 		(on_board yes)
 		(dnp no)
-		(property "Reference" "#PWR027"
+		(property "Reference" "#PWR021"
 			(at 74.93 78.74 0)
 			(effects
@@
 			(project "SteeringBoard"
 				(path "/1bc9055e-ec57-4cc6-8fa0-537b054d5f7c/2ae31cd1-3b20-41d6-acf0-8556f0359c18"
-					(reference "#PWR027")
+					(reference "#PWR021")
 					(unit 1)
 				)
@@
 		(dnp no)
 		(fields_autoplaced yes)
-		(property "Reference" "#PWR029"
+		(property "Reference" "#PWR023"
 			(at 154.94 87.63 0)
 			(effects
@@
 			(project "SteeringBoard"
 				(path "/1bc9055e-ec57-4cc6-8fa0-537b054d5f7c/2ae31cd1-3b20-41d6-acf0-8556f0359c18"
-					(reference "#PWR029")
+					(reference "#PWR023")
 					(unit 1)
 				)
@@
 		(on_board yes)
 		(dnp no)
-		(property "Reference" "R12"
+		(property "Reference" "R8"
 			(at 123.698 91.44 90)
 			(effects
@@
 			(project "SteeringBoard"
 				(path "/1bc9055e-ec57-4cc6-8fa0-537b054d5f7c/2ae31cd1-3b20-41d6-acf0-8556f0359c18"
-					(reference "R12")
+					(reference "R8")
 					(unit 1)
 				)
@@
 		(dnp no)
 		(fields_autoplaced yes)
-		(property "Reference" "#PWR030"
+		(property "Reference" "#PWR024"
 			(at 154.94 101.6 0)
 			(effects
@@
 			(project "SteeringBoard"
 				(path "/1bc9055e-ec57-4cc6-8fa0-537b054d5f7c/2ae31cd1-3b20-41d6-acf0-8556f0359c18"
-					(reference "#PWR030")
+					(reference "#PWR024")
 					(unit 1)
 				)
@@
 		(on_board yes)
 		(dnp no)
-		(property "Reference" "#PWR028"
+		(property "Reference" "#PWR022"
 			(at 74.93 93.98 0)
 			(effects
@@
 			(project "SteeringBoard"
 				(path "/1bc9055e-ec57-4cc6-8fa0-537b054d5f7c/2ae31cd1-3b20-41d6-acf0-8556f0359c18"
-					(reference "#PWR028")
+					(reference "#PWR022")
 					(unit 1)
 				)
@@
 		(on_board yes)
 		(dnp no)
-		(property "Reference" "C10"
+		(property "Reference" "C9"
 			(at 139.954 75.692 0)
 			(effects
@@
 			(project "SteeringBoard"
 				(path "/1bc9055e-ec57-4cc6-8fa0-537b054d5f7c/2ae31cd1-3b20-41d6-acf0-8556f0359c18"
-					(reference "C10")
+					(reference "C9")
 					(unit 1)
 				)
@@
 	(symbol
 		(lib_id "Jumper:Jumper_2_Open")
-		(at 120.65 99.06 0)
+		(at 120.65 97.79 0)
 		(unit 1)
 		(exclude_from_sim no)
@@
 		(dnp no)
 		(property "Reference" "JP1"
-			(at 120.65 97.028 0)
+			(at 120.65 95.758 0)
 			(effects
 				(font
@@
 		)
 		(property "Value" "Termination Resistors"
-			(at 120.65 101.6 0)
+			(at 120.65 100.33 0)
 			(effects
 				(font
@@
 		)
 		(property "Footprint" "Connector_PinHeader_2.54mm:PinHeader_1x02_P2.54mm_Vertical"
-			(at 120.65 99.06 0)
+			(at 120.65 97.79 0)
 			(effects
 				(font
@@
 		)
 		(property "Datasheet" "~"
-			(at 120.65 99.06 0)
+			(at 120.65 97.79 0)
 			(effects
 				(font
@@
 		)
 		(property "Description" "Jumper, 2-pole, open"
-			(at 120.65 99.06 0)
+			(at 120.65 97.79 0)
 			(effects
 				(font
@@
 		)
 		(property "PN" ""
-			(at 120.65 99.06 0)
+			(at 120.65 97.79 0)
 			(effects
 				(font
@@
 		)
 		(property "p/n" ""
-			(at 120.65 99.06 0)
-			(effects
-				(font
+			(at 120.65 97.79 0)
+			(effects
+				(font

Commit message: fixed the switch
Parts:
- renumbered R8 to R10
Changed lines of the file:
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@@
 		(on_board yes)
 		(dnp no)
-		(property "Reference" "#PWR021"
+		(property "Reference" "#PWR023"
 			(at 74.93 78.74 0)
 			(effects
@@
 			(project "SteeringBoard"
 				(path "/1bc9055e-ec57-4cc6-8fa0-537b054d5f7c/2ae31cd1-3b20-41d6-acf0-8556f0359c18"
-					(reference "#PWR021")
+					(reference "#PWR023")
 					(unit 1)
 				)
@@
 		(dnp no)
 		(fields_autoplaced yes)
-		(property "Reference" "#PWR023"
+		(property "Reference" "#PWR025"
 			(at 154.94 87.63 0)
 			(effects
@@
 			(project "SteeringBoard"
 				(path "/1bc9055e-ec57-4cc6-8fa0-537b054d5f7c/2ae31cd1-3b20-41d6-acf0-8556f0359c18"
-					(reference "#PWR023")
+					(reference "#PWR025")
 					(unit 1)
 				)
@@
 		(on_board yes)
 		(dnp no)
-		(property "Reference" "R8"
+		(property "Reference" "R10"
 			(at 123.698 91.44 90)
 			(effects
@@
 			(project "SteeringBoard"
 				(path "/1bc9055e-ec57-4cc6-8fa0-537b054d5f7c/2ae31cd1-3b20-41d6-acf0-8556f0359c18"
-					(reference "R8")
+					(reference "R10")
 					(unit 1)
 				)
@@
 		(dnp no)
 		(fields_autoplaced yes)
-		(property "Reference" "#PWR024"
+		(property "Reference" "#PWR026"
 			(at 154.94 101.6 0)
 			(effects
@@
 			(project "SteeringBoard"
 				(path "/1bc9055e-ec57-4cc6-8fa0-537b054d5f7c/2ae31cd1-3b20-41d6-acf0-8556f0359c18"
-					(reference "#PWR024")
+					(reference "#PWR026")
 					(unit 1)
 				)
@@
 		(on_board yes)
 		(dnp no)
-		(property "Reference" "#PWR022"
+		(property "Reference" "#PWR024"
 			(at 74.93 93.98 0)
 			(effects
@@
 			(project "SteeringBoard"
 				(path "/1bc9055e-ec57-4cc6-8fa0-537b054d5f7c/2ae31cd1-3b20-41d6-acf0-8556f0359c18"
-					(reference "#PWR022")
-					(unit 1)
-				)
+					(reference "#PWR024")
+					(unit 1)
+				)
