File: SteeringBoard.kicad_sch (KiCad schematic)
At the start: 30 parts, among them J1 SWD, J10 Conn_01x01_Pin, J11 Conn_01x01_Pin, J2 Conn_01x01_Pin, J3 Conn_01x01_Pin, J4 Conn_01x01_Pin, J5 Conn_01x01_Pin, J6 Conn_01x01_Pin, J7 Conn_01x01_Pin, J8 Conn_01x01_Pin, J9 Conn_01x01_Pin, SW1 Reset, U1 STM32L431CBTx

Commit message: scheme update
Parts:
- added D1, D2, D3, D4, D5: LED, LED_SMD:LED_0805_2012Metric, symbol Device:LED
- added J12, J13, J14, J15: Conn_01x01_Pin, Connector_PinHeader_2.54mm:PinHeader_1x01_P2.54mm_Vertical, symbol Connector:Conn_01x01_Pin
- added R1, R2, R4, R5, R6: 10k, Resistor_SMD:R_0805_2012Metric, symbol Device:R_US
- added R10, R11, R7, R8, R9: R_US, Resistor_SMD:R_0805_2012Metric, symbol Device:R_US
- J10, J11, J2, J3, J4, J5, J6, J7, J8, J9: footprint (none) -> Connector_PinHeader_2.54mm:PinHeader_1x01_P2.54mm_Vertical
- renumbered C5 to C3, C6 to C4, C7 to C5, C8 to C6, C9 to C7, C10 to C8
Connections:
- net CR_E+ is gone; now on net +3.3V: J8.1 (Pin_1)
- net RGEN_E+ is gone; now on net +3.3V: J6.1 (Pin_1)
- net +3.3V: now also J10.1 (Pin_1), J12.1 (Pin_1), J14.1 (Pin_1), R10.1, R11.1, R7.1, R8.1, R9.1
- net GND: now also D1.1 (K), D2.1 (K), D3.1 (K), D4.1 (K), D5.1 (K)
- net RGEN_E-: now also R1.1
- net at U1.13 (PA3): now also R5.2
- net at U1.14 (PA4): now also R6.2
- net REG-: now reaches J11.1 (Pin_1)
- net REG-: now also R4.1
- net CR_E- renamed CRS_SET-
- net CRS_SET-: now also R2.1
- net PA0: no longer names the net of U1.10 (PA0)
- net PA0: now also R1.2
- net PA1: no longer names the net of U1.11 (PA1)
- net PA1: now also R2.2
- net PA2: no longer names the net of U1.12 (PA2)
- net PA2: now also R4.2
- new net: D3.2 (A), R9.2
- new net: D2.2 (A), R8.2
- new net: D5.2 (A), R11.2
- new net: D1.2 (A), R7.2
- new net: D4.2 (A), R10.2
- new net HRN_PD-: J15.1 (Pin_1), R6.1
- new net TSS-: J13.1 (Pin_1), R5.1
- no-connect marks 10 -> 9
Other:
- moved on the sheet: FB2, U1

Commit message: layout changes
Parts:
- removed C4, C5: 100nF, Capacitor_SMD:C_0805_2012Metric, symbol Device:C
- added J16: Conn_01x02_Pin, UTSVT_Connectors:Molex_MicroFit3.0_1x2xP3.00mm_PolarizingPeg_Vertical, symbol Connector:Conn_01x02_Pin
- C1, C3, C6, C7, C8: footprint Capacitor_SMD:C_0805_2012Metric -> Capacitor_SMD:C_0603_1608Metric
- C2: value 100nF -> 300nF; footprint Capacitor_SMD:C_0805_2012Metric -> Capacitor_SMD:C_0603_1608Metric
- D1, D2, D3, D4, D5: footprint LED_SMD:LED_0805_2012Metric -> LED_SMD:LED_0603_1608Metric
- FB1, FB2: footprint Inductor_SMD:L_0805_2012Metric -> Inductor_SMD:L_0603_1608Metric
- J10, J11, J12, J13, J14, J15, J2, J3, J4, J5, J6, J7, J8, J9: footprint Connector_PinHeader_2.54mm:PinHeader_1x01_P2.54mm_Vertical -> TestPoint:TestPoint_Pad_D1.0mm
- R1, R10, R11, R2, R3, R4, R5, R6, R7, R8, R9: footprint Resistor_SMD:R_0805_2012Metric -> Resistor_SMD:R_0603_1608Metric
Connections:
- net CRS_SET-: now also R2.2, U1.11 (PA1); no longer R2.1
- net GND: now also R1.2, R2.1, R4.1, R5.1, R6.1
- net HRN_PD-: now also R6.2, U1.14 (PA4); no longer R6.1
- net REG-: now also R4.2, U1.12 (PA2); no longer R4.1
- net RGEN_E-: now also U1.10 (PA0)
- net TSS-: now also R5.2, U1.13 (PA3); no longer R5.1
- new net +12V: J16.2 (Pin_2)
- new net GNDPWR: J16.1 (Pin_1)
Other:
- moved on the sheet: R1, R2, R4, R5, R6

Commit message: board update
Parts:
- removed LOGO1: Dr. Hallock, UTSVT_Special:Hallock_Image_Tiny, symbol utsvt-misc:Logo_Placeholder
- removed LOGO2: UTSVT Logo, UTSVT_Special:UTSVT_Logo_Symbol, symbol utsvt-misc:Logo_Placeholder
- added J17: Conn_01x01_Pin, TestPoint:TestPoint_Pad_D1.0mm, symbol Connector:Conn_01x01_Pin
Connections:
- net 12V_Ext: now also J17.1 (Pin_1)
- net CAN_TX: now also U1.46 (PB9)
- net PB1: no longer names the net of U1.19 (PB1)
- net PB2: no longer names the net of U1.20 (PB2)
- net PB3: no longer names the net of U1.39 (PB3)
- net PB4: no longer names the net of U1.40 (PB4)
- net PB5: no longer names the net of U1.41 (PB5)
- no-connect marks 9 -> 29
Other:
- note removed: "Graphics/Logos"
- moved on the sheet: C1, C2, C3, C6, C7, C8, FB1, J1, R3, SW1

Commit message: board update
Parts:
- removed C3, C6, C8: 100nF, Capacitor_SMD:C_0603_1608Metric, symbol Device:C
- removed FB1, FB2: FerriteBead, Inductor_SMD:L_0603_1608Metric, symbol Device:FerriteBead
- removed J17: Conn_01x01_Pin, TestPoint:TestPoint_Pad_D1.0mm, symbol Connector:Conn_01x01_Pin
Connections:
- net VDD is gone; now on net +3.3V: R3.1
- net GNDA: no longer names the net of U1.8 (VSSA)
- net VDDA: no longer names the net of U1.9 (VDDA)
- no-connect marks 29 -> 31
Other:
- note removed: "VDDA Bypass Caps"
- note removed: "VDDA Seperation"

Commit message: finished board with ldo
Parts:
- removed J10, J11, J12, J13, J14, J15, J2, J3, J4, J5, J6, J7, J8, J9: Conn_01x01_Pin, TestPoint:TestPoint_Pad_D1.0mm, symbol Connector:Conn_01x01_Pin
- removed R1, R2, R4, R5, R6: 10k, Resistor_SMD:R_0603_1608Metric, symbol Device:R_US
- added C3, C4, C6, C7: 100nF, Capacitor_SMD:C_0603_1608Metric, symbol Device:C
- added D1: Heartbeat, LED_SMD:LED_0603_1608Metric, symbol Device:LED
- added J3: Conn_02x05_Counter_Clockwise, UTSVT_Connectors:CONN_SD-105310-100_10_MOL, symbol Connector_Generic:Conn_02x05_Counter_Clockwise
- added J4: Conn_01x04_Pin, NanoCONN:CONN_SD-105309-100_04_MOL, symbol Connector:Conn_01x04_Pin
- added R2: 2.2k, Resistor_SMD:R_0603_1608Metric, symbol Device:R
- C2: value 300nF -> 100nF
- renumbered C7 to C5, D1 to D2, D2 to D3, D3 to D4, D4 to D5, D5 to D6, J16 to J2, R3 to R1, R7 to R3, R8 to R4, R9 to R5, R10 to R6, R11 to R7
Connections:
- net +3.3V: now also U1.9 (VDDA), C3.1, C4.1, C6.1, C7.1, J3.1 (Pin_1), J3.2 (Pin_2), J3.3 (Pin_3), J3.4 (Pin_4), J3.5 (Pin_5); no longer R3.1, R4.1, R5.1, R6.1, R7.1
- net CAN_H: now also J4.1 (Pin_1)
- net CAN_L: now also J4.2 (Pin_2)
- net CAN_RX: now also J4.3 (Pin_3)
- net CAN_TX: now also J4.4 (Pin_4)
- net CRS_SET-: now also R4.1, U1.14 (PA4), J3.7 (Pin_7); no longer U1.11 (PA1)
- net GND: now also J1.2 (Pin_2), U1.8 (VSSA), C3.2, C4.2, C6.2, C7.2, D1.1 (K); no longer J1.3 (Pin_3)
- net HRN_PD-: now also R7.1, U1.17 (PA7), J3.10 (Pin_10); no longer U1.14 (PA4)
- net REG-: now also R5.1, U1.15 (PA5), J3.8 (Pin_8); no longer U1.12 (PA2)
- net RGEN_E-: now also R3.1, U1.13 (PA3), J3.6 (Pin_6); no longer U1.10 (PA0)
- net SWCLK: now also J1.4 (Pin_4), U1.34 (PA13); no longer J1.2 (Pin_2), U1.37 (PA14)
- net SWDIO: now also J1.3 (Pin_3), U1.33 (PA12); no longer J1.4 (Pin_4), U1.34 (PA13)
- net TSS-: now also R6.1, U1.16 (PA6), J3.9 (Pin_9); no longer U1.13 (PA3)
- new net: D1.2 (A), R2.2
- new net PA0: R2.1, U1.10 (PA0)
- no-connect marks 31 -> 28
Other:
- sheet PowerDist ports: added none; removed 12V_Ext
- note added: "VDDA Bypass Caps"
- moved on the sheet: D2, D3, D4, D5, D6, J2, R3, R4, R5, R6, R7

Commit message: final
Connections:
- net PA0: now also U1.25 (PB12); no longer U1.10 (PA0)
Changed lines of the file:
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@@
 	)
 	(no_connect
-		(at 97.79 88.9)
+		(at 97.79 86.36)
 	)
 	(no_connect
@@
 	)
 	(no_connect
-		(at 97.79 86.36)
+		(at 133.35 33.02)
 	)
 	(no_connect
@@
 		(pts
 			(xy 110.49 27.94) (xy 113.03 27.94)
+		)
+		(stroke
+			(width 0)
+			(type default)
+		)
+	)
+	(wire
+		(pts
+			(xy 92.71 88.9) (xy 97.79 88.9)
 		)
 		(stroke
@@
 	)
 	(label "PA0"
-		(at 133.35 33.02 0)
+		(at 92.71 88.9 180)
 		(fields_autoplaced yes)
 		(effects
@@
 				(size 1.27 1.27)
 			)
-			(justify left bottom)
-		)
-	)
+			(justify right bottom)
+		)
+	)

Commit message: fixed the switch
Parts:
- removed J3: Conn_02x05_Counter_Clockwise, UTSVT_Connectors:CONN_SD-105310-100_10_MOL, symbol Connector_Generic:Conn_02x05_Counter_Clockwise
- added D1, D8: LED, LED_SMD:LED_0603_1608Metric, symbol Device:LED
- added J2: Conn_02x06_Counter_Clockwise, UTSVT_Connectors:CONN_SD-105310-100_12_MOL, symbol Connector_Generic:Conn_02x06_Counter_Clockwise
- added R2, R9: R_US, Resistor_SMD:R_0603_1608Metric, symbol Device:R_US
- renumbered D1 to D2, D2 to D3, D3 to D4, D4 to D5, D5 to D6, D6 to D7, J2 to J3, J4 to J5, R2 to R3, R3 to R4, R4 to R5, R5 to R6, R6 to R7, R7 to R8
Connections:
- net +3.3V: now also J2.1 (Pin_1), J2.2 (Pin_2), J2.3 (Pin_3), J2.4 (Pin_4), J2.5 (Pin_5)
- net CRS_SET-: now also J2.9 (Pin_9)
- net GND: now also D1.1 (K), D8.1 (K)
- net HRN_PD-: now also J2.12 (Pin_12)
- net RGEN_E-: now also J2.8 (Pin_8)
- net TSSR-: now reaches U1.11 (PA1)
- net TSSR-: now also J2.6 (Pin_6), R2.1
- net TSSO-: now reaches U1.12 (PA2)
- net TSSO-: now also J2.7 (Pin_7), R9.1
- net REG- renamed CEN-
- net CEN-: now also J2.10 (Pin_10)
- net TSS- renamed TSSL-
- net TSSL-: now also J2.11 (Pin_11)
- new net: D8.2 (A), R9.2
- new net: D1.2 (A), R2.2
- no-connect marks 28 -> 26

Commit message: lo
Parts:
- renumbered J5 to J4
Connections:
- net GND: now also J1.3 (Pin_3); no longer J1.2 (Pin_2)
- net SWCLK: now also J1.2 (Pin_2); no longer J1.4 (Pin_4)
- net SWDIO: now also J1.4 (Pin_4); no longer J1.3 (Pin_3)
